Commit message: Make the IMU orientation a parameter, and fix the review findings
The IMU axis mapping was measured against one gimbal resting one way and then
written into the source. That is the wrong shape for a vendor-neutral driver:
the controller is a chip in a case, and which way that case is bolted into a
mount is a property of the build. imu_axis_map and imu_axis_sign now carry it,
defaulting to the board's own order passed through unchanged, and the README
explains how to measure the right values in about a minute without moving
anything. sbgc_description places gimbal_imu_link the same way, through
imu_parent / imu_xyz / imu_rpy.

A mapping that is not a permutation is refused with an error and the identity
used, because dropping or duplicating an axis still yields a plausible-looking
three-vector.

The review findings, most severe first:

Gyro calibration was cancelled by the driver's own control frames. The upstream
daemon documents that any CMD_CONTROL cancels a running calibration and
suppresses control for the whole of it; this sent one every 33 ms, so the board
aborted within a tick while the action went on to report success 4.5 s later.
It claimed a calibration that never happened. Control is now suppressed for the
duration, and the skip-settle path no longer ignores a failed send.

A cancelled trajectory called succeed(), which rclcpp_action permits only from
EXECUTING and otherwise throws - out of a timer callback, taking the process
with it. is_canceling() is now checked first.

An active trajectory re-submitted its target every cycle, so stop did not stick
and disarming left a goal that resumed on re-arming. Stop and disarm now end
what is in flight. Link loss no longer returns before the action ticks, which
had left their own link-unavailable checks unreachable.

Goals were accepted while the node was inactive, where no timer exists to
advance them; calibration could start beside a running trajectory; a second
trajectory silently displaced the first; and calibration counted a frozen
telemetry reading as "still", so a board that stopped answering could be
calibrated on evidence that had stopped arriving.

status.armed reported control_allowed && link_open rather than the arm bit, so
it stayed true after a successful disarm. on_shutdown and on_error left the
timers running over state that cleanup then destroyed.

auto_start:=false still configured the node and opened the serial port.
gimbal_imu_link was published but did not exist in any URDF. The description's
joint limits are now passed from the launch file so they can be given the same
numbers as the driver, and standalone.urdf.xacro forwards every macro argument
rather than accepting some and ignoring them.

FollowJointTrajectory now rejects goals carrying path_tolerance instead of
silently dropping the constraint: this server commands the final point and lets
the board slew, so it never observes the poses such a tolerance is defined
against. That reduction is documented rather than implied.

The README's multi-threaded safety claim was too broad. The lifecycle
transition callbacks touch the link and cannot join the port callback group.

Verified against a board 3.1 / firmware 2.63b0: the default mapping reads
+9.84 on z at rest, remapping to [2,1,0] with z inverted moves that reading to
x as expected, and an invalid map is refused in the log.

Co-Authored-By: Claude Opus 5 <noreply@anthropic.com>

File: sbgc_description/urdf/sbgc_gimbal.urdf.xacro (robot description, xacro)
@@ -18,5 +18,8 @@
       roll_min:=-0.785 roll_max:=0.785
       pitch_min:=-1.571 pitch_max:=0.698
-      max_rate:=0.79">
+      max_rate:=0.79
+      imu_parent:=pitch
+      imu_xyz:='0 0 0'
+      imu_rpy:='0 0 0'">
     <!-- Where the gimbal bolts to whatever carries it. -->
     <link name="${prefix}base_link">
@@ -89,4 +92,20 @@
       <limit lower="${pitch_min}" upper="${pitch_max}" effort="1.0" velocity="${max_rate}"/>
     </joint>
+    <!--
+      The controller's own IMU.
+      The driver publishes sensor_msgs/Imu in this frame, so it has to exist or
+      nothing can transform that data. Which link it rides on is a build
+      decision: on most mounts the board sits on the pitch stage with the
+      camera, but on some it is bolted to the base or the yaw stage instead.
+      imu_parent selects base, yaw, roll or pitch, and imu_xyz/imu_rpy place it
+      within that link, which is also where a board mounted at an angle is
+      described rather than by editing this file.
+    -->
+    <link name="${prefix}imu_link"/>
+    <joint name="${prefix}imu_joint" type="fixed">
+      <parent link="${prefix}${imu_parent}_link"/>
+      <child link="${prefix}imu_link"/>
+      <origin xyz="${imu_xyz}" rpy="${imu_rpy}"/>
+    </joint>
     <link name="${prefix}camera_link"/>
     <joint name="${prefix}camera_joint" type="fixed">

File: sbgc_description/urdf/standalone.urdf.xacro (robot description, xacro)
@@ -4,10 +4,37 @@
   without a robot around it. A real integration includes sbgc_gimbal.urdf.xacro
   from its own description and gives it a proper parent instead.
+  Every argument the macro takes is forwarded, so the bringup launch file can
+  pass the same joint limits it gives the driver. An argument declared here but
+  not forwarded would be accepted on the command line and silently ignored,
+  which is worse than not offering it.
 -->
 <robot name="sbgc_gimbal" xmlns:xacro="http://www.ros.org/wiki/xacro">
   <xacro:arg name="prefix" default="gimbal_"/>
+  <!-- Radians. Keep these in step with the driver's limit_min_deg /
+       limit_max_deg; robot_state_publisher will otherwise render joint
+       positions the driver refuses to command. -->
+  <xacro:arg name="roll_min"  default="-0.785"/>
+  <xacro:arg name="roll_max"  default="0.785"/>
+  <xacro:arg name="pitch_min" default="-1.571"/>
+  <xacro:arg name="pitch_max" default="0.698"/>
+  <xacro:arg name="yaw_min"   default="-2.967"/>
+  <xacro:arg name="yaw_max"   default="2.967"/>
+  <xacro:arg name="max_rate"  default="0.79"/>
+  <!-- Which stage the controller is bolted to, and where on it. -->
+  <xacro:arg name="imu_parent" default="pitch"/>
+  <xacro:arg name="imu_xyz"    default="0 0 0"/>
+  <xacro:arg name="imu_rpy"    default="0 0 0"/>
   <xacro:include filename="$(find sbgc_description)/urdf/sbgc_gimbal.urdf.xacro"/>
   <link name="base_link"/>
-  <xacro:sbgc_gimbal prefix="$(arg prefix)" parent="base_link">
+  <xacro:sbgc_gimbal
+      prefix="$(arg prefix)"
+      parent="base_link"
+      roll_min="$(arg roll_min)"   roll_max="$(arg roll_max)"
+      pitch_min="$(arg pitch_min)" pitch_max="$(arg pitch_max)"
+      yaw_min="$(arg yaw_min)"     yaw_max="$(arg yaw_max)"
+      max_rate="$(arg max_rate)"
+      imu_parent="$(arg imu_parent)"
+      imu_xyz="$(arg imu_xyz)"
+      imu_rpy="$(arg imu_rpy)">
     <origin xyz="0 0 0" rpy="0 0 0"/>
   </xacro:sbgc_gimbal>
